File: Elevador-Aço-UFES-2017/Elevador-Aço-UFES-2017.sch (KiCad schematic (older format))
At the start: 62 parts, among them Q1 TIP126, Q2 TIP126, Q3 TIP121, Q4 TIP121, U1 74HC14, U2 PHOTODIODE, U3 LM7805, U4 7406

Commit message: atualizando
Parts:
- B1, B2, B3, B4, B5, B6: symbol SW_PUSH -> Elevador-Aço-UFES-2017-rescue:SW_PUSH
- C_Branco, C_Laranja_1, C_Laranja_2: symbol C -> Elevador-Aço-UFES-2017-rescue:C
- D1, D2, D3, D4, D5, D6, D7, D8: symbol LED -> Elevador-Aço-UFES-2017-rescue:LED
- D? (x4): symbol D -> Elevador-Aço-UFES-2017-rescue:D
- MOTOR, R1, R10, R11, R12, R13, R2, R3, R4, R5, R6, R7, R8, R9, R? (x14): symbol R -> Elevador-Aço-UFES-2017-rescue:R
- P?: symbol CONN_02X13 -> Elevador-Aço-UFES-2017-rescue:CONN_02X13
- Q1, Q2: symbol TIP126 -> Elevador-Aço-UFES-2017-rescue:TIP126
- Q3, Q4: symbol TIP121 -> Elevador-Aço-UFES-2017-rescue:TIP121
- U1: symbol 74HC14 -> Elevador-Aço-UFES-2017-rescue:74HC14
- U2: symbol PHOTODIODE -> Elevador-Aço-UFES-2017-rescue:PHOTODIODE
- U3: symbol LM7805 -> Elevador-Aço-UFES-2017-rescue:LM7805
- U4, U? (x4): symbol 74LS05 -> Elevador-Aço-UFES-2017-rescue:74LS05
