File: Elevador-Aço-UFES-2017/Conector/Conector do Elevador-UFES-2017.sch (KiCad schematic (older format))
At the start: 9 parts, among them J1 DB25, P1 CONN_01X04, P2 CONN_01X04, P3 CONN_01X04, P4 CONN_01X04, P5 CONN_01X04, P6 CONN_01X04, P7 CONN_01X08

Commit message: atualizando
Parts:
- ALB1: symbol ALB -> Conector-do-Elevador-UFES-2017-rescue:ALB
- J1: symbol DB25 -> Conector-do-Elevador-UFES-2017-rescue:DB25
- P1, P2, P3, P4, P5, P6: symbol CONN_01X04 -> Conector-do-Elevador-UFES-2017-rescue:CONN_01X04
- P7: symbol CONN_01X08 -> Conector-do-Elevador-UFES-2017-rescue:CONN_01X08
Changed lines of the file:
@@
-EESchema Schematic File Version 2
-LIBS:power
-LIBS:device
-LIBS:transistors
-LIBS:conn
-LIBS:linear
-LIBS:regul
-LIBS:74xx
-LIBS:cmos4000
-LIBS:adc-dac
-LIBS:memory
-LIBS:xilinx
-LIBS:microcontrollers
-LIBS:dsp
-LIBS:microchip
-LIBS:analog_switches
-LIBS:motorola
-LIBS:texas
-LIBS:intel
-LIBS:audio
-LIBS:interface
-LIBS:digital-audio
-LIBS:philips
-LIBS:display
-LIBS:cypress
-LIBS:siliconi
-LIBS:opto
-LIBS:atmel
-LIBS:contrib
-LIBS:valves
-LIBS:alb
+EESchema Schematic File Version 4
 LIBS:Conector do Elevador-UFES-2017-cache
-EELAYER 25 0
+EELAYER 26 0
 EELAYER END
 $Descr A4 11693 8268
@@
 $EndDescr
 $Comp
-L DB25 J1
+L Conector-do-Elevador-UFES-2017-rescue:DB25 J1
 U 1 1 59CF9F73
 P 2300 2900
@@
 Conexão Placa do elevador\n
 $Comp
-L CONN_01X04 P2
+L Conector-do-Elevador-UFES-2017-rescue:CONN_01X04 P2
 U 1 1 5A0B70BC
 P 4400 1800
@@
 $EndComp
 $Comp
-L CONN_01X04 P3
+L Conector-do-Elevador-UFES-2017-rescue:CONN_01X04 P3
 U 1 1 5A0B7120
 P 4400 2300
@@
 $EndComp
 $Comp
-L CONN_01X04 P4
+L Conector-do-Elevador-UFES-2017-rescue:CONN_01X04 P4
 U 1 1 5A0B715A
 P 4400 2800
@@
 $EndComp
 $Comp
-L CONN_01X04 P5
+L Conector-do-Elevador-UFES-2017-rescue:CONN_01X04 P5
 U 1 1 5A0B7185
 P 4400 3350
@@
 $EndComp
 $Comp
-L CONN_01X04 P6
+L Conector-do-Elevador-UFES-2017-rescue:CONN_01X04 P6
 U 1 1 5A0B71A6
 P 4400 3850
@@
 	3200 1950 4200 1950
 Wire Wire Line
-	2750 4000 4200 4000
+	2750 4000 4150 4000
 Wire Wire Line
 	2750 3200 3100 3200
@@
 	3000 3600 3000 3900
 Wire Wire Line
-	3000 3900 4200 3900
-Wire Wire Line
 	2750 3400 2900 3400
 Wire Wire Line
 	2900 3400 2900 3800
 Wire Wire Line
-	2900 3800 4200 3800
+	2900 3800 3900 3800
 Wire Wire Line
 	3100 3200 3100 3700
 Wire Wire Line
-	3100 3700 4200 3700
-Wire Wire Line
 	2750 4100 3700 4100
 Wire Wire Line
@@
 	3700 3500 4200 3500
 Wire Wire Line
-	2750 3900 3450 3900
-Wire Wire Line
 	3450 3900 3450 3400
 Wire Wire Line
 	3450 3400 4200 3400
 Wire Wire Line
-	2750 3700 3250 3700
-Wire Wire Line
-	3250 3700 3250 3300
-Wire Wire Line
-	3250 3300 4200 3300
-Wire Wire Line
 	2750 3500 3250 3500
 Wire Wire Line
-	3250 3500 3250 3200
-Wire Wire Line
 	3250 3200 4200 3200
 Wire Wire Line
-	2750 3300 3450 3300
-Wire Wire Line
 	3450 3300 3450 2950
 Wire Wire Line
@@
 	4200 2300 4200 2250
 $Comp
-L CONN_01X04 P1
+L Conector-do-Elevador-UFES-2017-rescue:CONN_01X04 P1
 U 1 1 5A0B79B7
 P 3600 2550
@@
 	3350 2600 3400 2600
 $Comp
-L ALB ALB1
+L Conector-do-Elevador-UFES-2017-rescue:ALB ALB1
 U 1 1 5A0B781C
 P 2600 4550
@@
 $EndComp
 $Comp
-L CONN_01X08 P7
+L Conector-do-Elevador-UFES-2017-rescue:CONN_01X08 P7
 U 1 1 5A0E0FAE
 P 4050 4550
@@
 	4150 4100 4150 4000
 Connection ~ 4150 4000
+Wire Wire Line
+	3650 3700 4200 3700
+Wire Wire Line
+	3900 3800 4200 3800
+Wire Wire Line
+	4100 3900 4200 3900
+Wire Wire Line
+	4150 4000 4200 4000
+Wire Wire Line
+	2750 3900 4100 3900
+Wire Wire Line
+	2750 3700 3650 3700
+Wire Wire Line
+	3250 3200 3250 3700
+Wire Wire Line
+	2750 3300 4200 3300
 $EndSCHEMATC
