File: Elevador-Aço-UFES-2017/Conector/Conector Controlador + fonte/Conector Controlador + fonte.sch (KiCad schematic (older format))
At the start: 8 parts, among them J1 DB25, P1 CONN_01X04, P2 CONN_01X08, P3 CONN_01X04, P4 CONN_01X04, P5 CONN_01X04, P6 CONN_01X04

Commit message: atualizando
Parts:
- J1: symbol DB25 -> Conector-Controlador-+-fonte-rescue:DB25
- P1, P3, P4, P5, P6, botões1: symbol CONN_01X04 -> Conector-Controlador-+-fonte-rescue:CONN_01X04
- P2: symbol CONN_01X08 -> Conector-Controlador-+-fonte-rescue:CONN_01X08
Changed lines of the file:
@@
-EESchema Schematic File Version 2
-LIBS:power
-LIBS:device
-LIBS:transistors
-LIBS:conn
-LIBS:linear
-LIBS:regul
-LIBS:74xx
-LIBS:cmos4000
-LIBS:adc-dac
-LIBS:memory
-LIBS:xilinx
-LIBS:microcontrollers
-LIBS:dsp
-LIBS:microchip
-LIBS:analog_switches
-LIBS:motorola
-LIBS:texas
-LIBS:intel
-LIBS:audio
-LIBS:interface
-LIBS:digital-audio
-LIBS:philips
-LIBS:display
-LIBS:cypress
-LIBS:siliconi
-LIBS:opto
-LIBS:atmel
-LIBS:contrib
-LIBS:valves
+EESchema Schematic File Version 4
 LIBS:Conector Controlador + fonte-cache
-EELAYER 25 0
+EELAYER 26 0
 EELAYER END
 $Descr A4 11693 8268
@@
 $EndDescr
 $Comp
-L DB25 J1
+L Conector-Controlador-+-fonte-rescue:DB25 J1
 U 1 1 59CF9F73
 P 2300 2900
@@
 Conexão Placa  Controlador + Fonte\n
 $Comp
-L CONN_01X04 botões1
+L Conector-Controlador-+-fonte-rescue:CONN_01X04 botões1
 U 1 1 5A0E1311
 P 4550 1750
@@
 $EndComp
 $Comp
-L CONN_01X04 P1
+L Conector-Controlador-+-fonte-rescue:CONN_01X04 P1
 U 1 1 5A0E158A
 P 3400 2600
@@
 $EndComp
 $Comp
-L CONN_01X04 P4
+L Conector-Controlador-+-fonte-rescue:CONN_01X04 P4
 U 1 1 5A0E15A9
 P 4550 2300
@@
 $EndComp
 $Comp
-L CONN_01X04 P5
+L Conector-Controlador-+-fonte-rescue:CONN_01X04 P5
 U 1 1 5A0E15D4
 P 4550 3000
@@
 $EndComp
 $Comp
-L CONN_01X04 P6
+L Conector-Controlador-+-fonte-rescue:CONN_01X04 P6
 U 1 1 5A0E15FD
 P 4550 3600
@@
 $EndComp
 $Comp
-L CONN_01X04 P3
+L Conector-Controlador-+-fonte-rescue:CONN_01X04 P3
 U 1 1 5A0E1688
 P 4400 4100
@@
 $EndComp
 $Comp
-L CONN_01X08 P2
+L Conector-Controlador-+-fonte-rescue:CONN_01X08 P2
 U 1 1 5A0E16AD
 P 3500 4700
@@
 	3250 4000 3250 4250
 Wire Wire Line
-	3250 4250 4200 4250
+	3250 4250 3750 4250
 Wire Wire Line
 	2750 4100 3850 4100
@@
 	3900 3550 4350 3550
 Wire Wire Line
-	2750 3200 3700 3200
+	2750 3200 3150 3200
 Wire Wire Line
 	3700 3200 3700 3950
@@
 	3700 3950 4200 3950
 Wire Wire Line
-	2750 3400 3450 3400
+	2750 3400 3400 3400
 Wire Wire Line
 	3450 3400 3450 4050
@@
 	3350 3600 3350 4150
 Wire Wire Line
-	3350 4150 4200 4150
+	3350 4150 3550 4150
 Wire Wire Line
 	3150 4500 3150 3200
@@
 Text Notes 4700 4300 0    60   ~ 0
 21\n22\n23\n25
+Wire Wire Line
+	3150 3200 3700 3200
+Wire Wire Line
+	3400 3400 3450 3400
+Wire Wire Line
+	3550 4150 4200 4150
+Wire Wire Line
+	3750 4250 4200 4250
 $EndSCHEMATC
